Commit message: added low res model & plannar movement

File: description/gazebo_control.xacro (robot description, xacro)
@@ -1,3 +1,13 @@
 <?xml version="1.0"?>
 <robot xmlns:xacro="http://www.ros.org/wiki/xacro">
+	<gazebo>
+		<plugin name="holonomic_control" filename="libgazebo_ros_planar_move.so">
+      		<commandTopic>cmd_vel</commandTopic>
+      		<odometryTopic>odom</odometryTopic>
+      		<odometryFrame>odom</odometryFrame>
+      		<odometryRate>20.0</odometryRate>
+      		<robotBaseFrame>base_link</robotBaseFrame>
+			<publishTF>true</publishTF>
+    	</plugin>
+  </gazebo>
 </robot>

File: description/robot_core.xacro (robot description, xacro)
@@ -6,14 +6,149 @@
     </material>
     <material name="orange">
-	<color rgba="1 0.3 0.1 1"/>
+		<color rgba="1 0.3 0.1 1"/>
     </material>
     <material name="blue">
-	<color rgba="0.2 0.2 1 1"/>
+		<color rgba="0.2 0.2 1 1"/>
     </material>
     <material name="black">
-	<color rgba="0 0 0 1"/>
+		<color rgba="0 0 0 1"/>
     </material>
     <!-- BASE LINK -->
     <link name="base_link">
     </link>
+    <!-- CHASSIS LINK -->
+	<joint name="chassis_joint" type="fixed">
+		<parent link="base_link"/>
+		<child link="chassis"/>
+		<origin xyz="0 0 0"/>
+	</joint>
+	<link name="chassis">
+		<visual>
+			<origin xyz="0 0 0.1"/>
+			<geometry>
+				<box size="0.5 0.5 0.03"/>
+			</geometry>
+			<material name="white"/>
+		</visual>
+		<collision>
+			<origin xyz="0 0 0.1"/>
+			<geometry>
+				<box size="0.5 0.5 0.03"/>
+			</geometry>
+		</collision>
+		<xacro:inertial_box mass="0.2" x="0.5" y="0.5" z="0.03">
+        	<origin xyz="0 0 0.1" rpy="0 0 0"/>
+    	</xacro:inertial_box>
+	</link>
+	<gazebo reference="chassis">
+        <material>Gazebo/White</material>
+    </gazebo>
+	<!-- WHEEL1 LINK -->
+	<joint name="wheel1_joint" type="continuous">
+		<parent link="base_link"/>
+		<child link="wheel1_link"/>
+		<origin xyz="0 0.27 0.08" rpy="-${pi/2} 0 0"/>
+		<axis xyz="0 0 1"/>
+	</joint>
+	<link name="wheel1_link">
+		<visual>
+			<geometry>
+				<cylinder radius="0.08" length="0.04"/>
+			</geometry>
+		</visual>
+		<collision>
+			<geometry>
+				<cylinder radius="0.08" length="0.04"/>
+			</geometry>
+		</collision>
+		<xacro:inertial_cylinder mass="0.1" length="0.4" radius="0.8">
+        	<origin xyz="0 0 0" rpy="0 0 0"/>
+    	</xacro:inertial_cylinder>
+	</link>
+	<gazebo reference="wheel1_link">
+        <material>Gazebo/Black</material>
+		<mu1 value="0.5"/>
+		<mu2 value="0.5"/>
+    </gazebo>
+	<!-- WHEEL2 LINK -->
+	<joint name="wheel2_joint" type="continuous">
+		<parent link="base_link"/>
+		<child link="wheel2_link"/>
+		<origin xyz="0 -0.27 0.08" rpy="${pi/2} 0 0"/>
+		<axis xyz="0 0 -1"/>
+	</joint>
+	<link name="wheel2_link">
+		<visual>
+			<geometry>
+				<cylinder radius="0.08" length="0.04"/>
+			</geometry>
+		</visual>
+		<collision>
+			<geometry>
+				<cylinder radius="0.08" length="0.04"/>
+			</geometry>
+		</collision>
+		<xacro:inertial_cylinder mass="0.1" length="0.4" radius="0.8">
+        	<origin xyz="0 0 0" rpy="0 0 0"/>
+    	</xacro:inertial_cylinder>
+	</link>
+	<gazebo reference="wheel2_link">
+        <material>Gazebo/Black</material>
+		<mu1 value="0.5"/>
+		<mu2 value="0.5"/>
+    </gazebo>
+	<!-- WHEEL3 LINK -->
+	<joint name="wheel3_joint" type="continuous">
+		<parent link="base_link"/>
+		<child link="wheel3_link"/>
+		<origin xyz="0.27 0 0.08" rpy="${-pi/2} 0 ${-pi/2}"/>
+		<axis xyz="0 0 1"/>
+	</joint>
+	<link name="wheel3_link">
+		<visual>
+			<geometry>
+				<cylinder radius="0.08" length="0.04"/>
+			</geometry>
+		</visual>
+		<collision>
+			<geometry>
+				<cylinder radius="0.08" length="0.04"/>
+			</geometry>
+		</collision>
+		<xacro:inertial_cylinder mass="0.1" length="0.4" radius="0.8">
+        	<origin xyz="0 0 0" rpy="0 0 0"/>
+    	</xacro:inertial_cylinder>
+	</link>
+	<gazebo reference="wheel3_link">
+        <material>Gazebo/Black</material>
+		<mu1 value="0.5"/>
+		<mu2 value="0.5"/>
+    </gazebo>
+	<!-- WHEEL4 LINK -->
+	<joint name="wheel4_joint" type="continuous">
+		<parent link="base_link"/>
+		<child link="wheel4_link"/>
+		<origin xyz="-0.27 0 0.08" rpy="${pi/2} 0 ${-pi/2}"/>
+		<axis xyz="0 0 -1"/>
+	</joint>
+	<link name="wheel4_link">
+		<visual>
+			<geometry>
+				<cylinder radius="0.08" length="0.04"/>
+			</geometry>
+		</visual>
+		<collision>
+			<geometry>
+				<cylinder radius="0.08" length="0.04"/>
+			</geometry>
+		</collision>
+		<xacro:inertial_cylinder mass="0.1" length="0.4" radius="0.8">
+        	<origin xyz="0 0 0" rpy="0 0 0"/>
+    	</xacro:inertial_cylinder>
+	</link>
+	<gazebo reference="wheel4_link">
+        <material>Gazebo/Black</material>
+		<mu1 value="0.5"/>
+		<mu2 value="0.5"/>
+    </gazebo>
 </robot>
